File: new_rs422_module_kicad.kicad_pcb (KiCad board)
At the start: 2 copper layers, 50 x 31.8 mm, 26 parts, among them J1 DS1037-01-09FNAKSI74, J2 Conn_01x04, Q1 BC847, U1 MAX490E

Commit message: done & gerbers generated
Parts:
- moved C1 1.27 mm to (37.8, 38.3)
Connections:
- J1 pad 4: Net-(J1-Pad4) -> DSUB_RS422_B
- J1 pad 5: Net-(J1-Pad5) -> DSUB_RS422_A
- J1 pad 8: Net-(J1-Pad8) -> DSUB_RS422_Y
- J1 pad 9: Net-(J1-Pad9) -> DSUB_RS422_Z
- Q1 pad 3: Net-(Q1-Pad3) -> PHOTOMETER_RX
- R1 pad 1: Net-(Q1-Pad3) -> PHOTOMETER_RX
- R9 pad 2: Net-(R9-Pad2) -> PHOTOMETER_TX
- U1 pad 3: Net-(R9-Pad2) -> PHOTOMETER_TX
Routing:
- net GND: track 0.00 -> 36.4 mm, vias 0 -> 5
- net DSUB_RS422_A: track 0.00 -> 32.6 mm, vias 0 -> 1
- net DSUB_RS422_Y: track 0.00 -> 28.3 mm
- net DSUB_RS422_Z: track 0.00 -> 27.4 mm
- net DSUB_RS422_B: track 0.00 -> 26.1 mm
- net Net-(R11-Pad2): track 0.00 -> 24.1 mm
- net PHOTOMETER_TX: track 0.00 -> 22.0 mm, vias 0 -> 2
- net PHOTOMETER_RX: track 0.00 -> 11.4 mm
- net Net-(R3-Pad2): track 0.00 -> 7.20 mm
- net Net-(R4-Pad2): track 0.00 -> 7.20 mm
- net Net-(Q1-Pad1): track 0.00 -> 6.14 mm
- net Net-(JP2-Pad1): track 0.00 -> 5.35 mm
- net Net-(JP1-Pad1): track 0.00 -> 5.35 mm
- net Net-(D1-Pad1): track 0.00 -> 5.11 mm
- net Net-(R5-Pad2): track 0.00 -> 4.38 mm
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- added copper zone on F.Cu, net +5V
- added copper zone on B.Cu, net GND
Other:
- board text added: "+5V"
- board text added: "GND"
- board text added: "RX"
- board text added: "TX"
- board text added: "Water Minilab RS422 module"
- board text removed: "APA/ANYA CSATLAKOZÓ???"
