File: new_rs422_module_kicad.sch (KiCad schematic (older format))
At the start: 26 parts, among them J1 DS1037-01-09FNAKSI74, J2 Conn_01x04, Q1 BC847, U1 MAX490E

Commit message: done & gerbers generated
Connections:
- net DSUB_RS422_A: now also J1.5
- net DSUB_RS422_B: now also J1.4
- net DSUB_RS422_Y: now also J1.8
- net DSUB_RS422_Z: now also J1.9
- net PHOTOMETER_RX: now also Q1.3 (C), R1.1
- net PHOTOMETER_TX: now also R9.2, U1.3 (DI)
Other:
- moved on the sheet: C1, C2, D1, J1, R10
